File: PCB/FireFly.kicad_pcb (KiCad board)
At the start: 2 copper layers, 112 x 24 mm, 86 parts, among them Q1 LED_RGB 5050, Q2 MMBT2222, SW1 BUTTON, SW2 SWITCH, SW3 BUTTON

Commit message: v1 sent to factory
Parts:
- removed C15, C32: 100pF, Capacitors:CAP_0402
- removed C16, C20: *, Capacitors:CAP_0402
- removed L5: *, Inductors:IND_0402
- removed RP3, RP4: REFPOINT, PCB:REF_POINT_1MM
- ANT1: footprint Antennas:LcktSnd_868 -> Antennas:Firefly_2400
- ANT2: footprint Antennas:LcktSnd_2d41 -> Antennas:Firefly_868
- C14, C17, C2, C21, C22, C23, C24, C26, C27, C28, C29, C3, C30, C31, C9: footprint Capacitors:CAP_0603 -> Capacitors:CAP_0402
- XL1: footprint Connectors:PLD-8 -> Connectors:PLD-8_LOCK; moved to F.Cu
- XL2: value CONN_5 -> CONN_4; footprint Connectors:PLS-5 -> Connectors:PLS-4
- moved C19 90.2 mm to (174.4, 95.4), turned to 180 degrees
- moved L2 87.8 mm to (165.7, 90.7), turned to 90 degrees
- moved C6 85.7 mm to (163.8, 84.6), turned to 90 degrees
- moved C8 84.7 mm to (164.1, 90.7), turned to 270 degrees
- moved L8 84.0 mm to (120.3, 98.3)
- moved XTAL3 83.0 mm to (127.0, 90.1), turned to 180 degrees
- moved XTAL1 82.9 mm to (161.4, 95.0), turned to 90 degrees
- moved C34 82.8 mm to (119.8, 96.6), turned to 90 degrees
- moved HOLE4 82.6 mm to (121.4, 82.2)
- moved C29 82.1 mm to (127.1, 92.8)
- moved C4 81.9 mm to (170.8, 91.3), turned to 270 degrees
- moved RP1 81.6 mm to (125.0, 81.7)
- moved C23 81.6 mm to (124.3, 90.1), turned to 90 degrees
- moved R1 81.4 mm to (157.7, 91.2), turned to 90 degrees
- moved C30 80.5 mm to (132.1, 96.6)
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Connections:
- ANT1 pad 1: Net-(ANT1-Pad1) -> /RF2400
- C33 pad 1: Net-(C32-Pad1) -> /RF3
- DD2 pad 41: /P29 -> /VDD_NRF
- L3 pad 2: Net-(C15-Pad1) -> /RF2400
- L8 pad 2: Net-(C32-Pad1) -> /RF3
- XL1 pad 2: /NRF_SWCLK -> /NRF_SWDIO
- XL1 pad 4: /NRF_SWDIO -> /NRF_SWCLK
- XL1 pad 7: /NRF_NRST -> /NRF_SWO
- XL1 pad 8: /NRF_SWO -> /NRF_NRST
Routing:
- net GND: track 0.00 -> 274.7 mm, vias 0 -> 100
- net +BATT: track 0.00 -> 98.6 mm, vias 0 -> 3
- net VCC: track 0.00 -> 57.5 mm, vias 0 -> 5
- net /BTN1: track 0.00 -> 45.8 mm
- net /NRF_DBG_RX: track 0.00 -> 45.5 mm, vias 0 -> 1
- net /CC_GDO2: track 0.00 -> 43.9 mm, vias 0 -> 4
- net /LED_EN: track 0.00 -> 42.6 mm, vias 0 -> 2
- net /CC_CS: track 0.00 -> 41.3 mm, vias 0 -> 2
- net /SDA_PILL: track 0.00 -> 39.4 mm, vias 0 -> 1
- net /NRF_DBG_TX: track 0.00 -> 39.0 mm, vias 0 -> 1
- net /CC_MOSI: track 0.00 -> 38.6 mm, vias 0 -> 2
- net /CC_GDO0: track 0.00 -> 38.5 mm, vias 0 -> 2
- net /CC_MISO: track 0.00 -> 37.9 mm, vias 0 -> 2
- net /CC_SCK: track 0.00 -> 37.9 mm, vias 0 -> 2
- net /NRF_SWDIO: track 0.00 -> 37.0 mm, vias 0 -> 1
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- added copper zone on B.Cu, net GND
- added copper zone on F.Cu, net GND
Other:
- outline, holes or cut-outs redrawn
- net class Default: clearance 0.2 -> 0.15; trace_width 0.25 -> 0.15; via_dia 0.8 -> 0.7; via_drill 0.4 -> 0.3
- net class RF2400 added: clearance 0.2, trace_width 1.1, via_dia 0.7, via_drill 0.3
- net class Wide added: clearance 0.2, trace_width 0.5, via_dia 0.7, via_drill 0.3
- rule pad_to_mask_clearance: 0.051 -> 0.1
- rule solder_mask_min_width: 0.25 -> 0.15
- rule trace_clearance: 0.2 -> 0.15
- rule trace_min: 0.2 -> 0.125
- board text added: "Buzzer"
- board text added: "EE"
- board text added: "LED"
- board text added: "Ostranna Firefly v1"
- board text added: "Pill"
- board text added: "Radio 868 MHz"

Commit message: Preparing for production
Parts:
- added D2: BAT54WS, Diodes:SOD323, F.Cu at (184.2, 83.8)
- BZ1: value PS-9627 -> KLJ-09650-3027
- C33: value * -> DoNotMount
- C34: value * -> 2.7pF
- L8: value * -> 8.2nH
Connections:
- DA1 pad 3: (no net) -> Net-(DA1-Pad3)
- DD2 pad 11: (no net) -> Net-(DD2-Pad11)
- DD2 pad 12: (no net) -> Net-(DD2-Pad12)
- DD2 pad 32: (no net) -> Net-(DD2-Pad32)
- DD2 pad 44: (no net) -> Net-(DD2-Pad44)
- SW2 pad 3: (no net) -> Net-(SW2-Pad3)

Commit message: PCB v1.1
Parts:
- B1: footprint Installation:BATTERY_AAA_X2 -> Installation:BATTERY_AAA_X2_PLUS_LEFT
- BZ1: footprint Installation:BUZZER_HC0903 -> Installation:BUZZER_KLJ-09650-3027
- moved D2 4.78 mm to (183.2, 88.5)
- moved Q2 0.50 mm to (178.8, 86.7)
- moved C12 0.22 mm to (176.6, 95.6)
- moved C19 0.22 mm to (174.5, 95.6)
- moved R10 0.10 mm to (176.3, 86.7)
Connections:
- DA1 pad 3: Net-(DA1-Pad3) -> (no net)
- DD2 pad 11: Net-(DD2-Pad11) -> (no net)
- DD2 pad 12: Net-(DD2-Pad12) -> (no net)
- DD2 pad 32: Net-(DD2-Pad32) -> (no net)
- DD2 pad 44: Net-(DD2-Pad44) -> (no net)
- SW2 pad 3: Net-(SW2-Pad3) -> (no net)
Routing:
- net VCC: track 57.5 -> 60.4 mm
- net /BuzzerOut: track 2.22 -> 4.19 mm
- net /RF2400: track 6.99 -> 8.29 mm
- net /NRF_SWDIO: track 37.0 -> 35.7 mm
- net GND: track 274.7 -> 275.6 mm
- net /BAT_IN: track 6.73 -> 7.68 mm
- net /NRF_SWCLK: track 34.2 -> 33.3 mm
- net Net-(C12-Pad2): track 6.19 -> 7.04 mm
- net /NRF_NRST: track 31.6 -> 30.9 mm
- net /NRF_SWO: track 33.4 -> 32.9 mm
Other:
- board text added: "Ostranna Firefly v1.1"
- board text removed: "Ostranna Firefly v1"
